File: MotorBoardPrototyp4_polyfuse.brd (EAGLE design)
At the start: 85 x 56 mm, 88 parts, among them IC1 OPA4340E, IC2 OPA4340E

Commit message: corrected MISO and MOSI closes #2
Connections:
- net DIN: now also PCB1.19; no longer PCB1.21
- net DOUT: now also PCB1.21; no longer PCB1.19
Routing:
- net DIN: track 26.1 -> 15.1 mm, vias 1 -> 0
- net DOUT: track 14.0 -> 16.4 mm
Changed lines of the file:
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@@
 <setting verticaltext="up"/>
 </settings>
-<grid distance="0.025" unitdist="inch" unit="inch" style="lines" multiple="1" display="yes" altdistance="0.00125" altunitdist="mil" altunit="mil"/>
+<grid distance="0.0125" unitdist="inch" unit="inch" style="lines" multiple="1" display="yes" altdistance="0.00125" altunitdist="mil" altunit="mil"/>
 <layers>
 <layer number="1" name="Top" color="4" fill="1" visible="yes" active="yes"/>
@@
 <signal name="DIN">
 <contactref element="U$58" pad="11"/>
-<contactref element="PCB1" pad="21"/>
-<wire x1="20.0025" y1="44.6659" x2="20.0025" y2="42.545" width="0.254" layer="16"/>
-<wire x1="20.0025" y1="42.545" x2="21.59" y2="40.9575" width="0.254" layer="16"/>
-<wire x1="21.59" y1="40.9575" x2="30.48" y2="40.9575" width="0.254" layer="16"/>
-<wire x1="30.48" y1="40.9575" x2="35.2425" y2="45.72" width="0.254" layer="16"/>
-<via x="35.2425" y="45.72" extent="1-16" drill="0.35"/>
-<wire x1="35.2425" y1="45.72" x2="35.2425" y2="49.7575" width="0.254" layer="1"/>
-<wire x1="35.2425" y1="49.7575" x2="33.77" y2="51.23" width="0.254" layer="1"/>
+<contactref element="PCB1" pad="19"/>
+<wire x1="20.0025" y1="44.6659" x2="20.0025" y2="46.6725" width="0.254" layer="16"/>
+<wire x1="20.0025" y1="46.6725" x2="22.86" y2="49.53" width="0.254" layer="16"/>
+<wire x1="22.86" y1="49.53" x2="29.53" y2="49.53" width="0.254" layer="16"/>
+<wire x1="29.53" y1="49.53" x2="31.23" y2="51.23" width="0.254" layer="16"/>
 </signal>
 <signal name="DOUT">
 <contactref element="U$58" pad="12"/>
-<contactref element="PCB1" pad="19"/>
-<wire x1="21.2725" y1="44.6659" x2="21.2725" y2="46.99" width="0.254" layer="16"/>
-<wire x1="21.2725" y1="46.99" x2="23.495" y2="49.2125" width="0.254" layer="16"/>
-<wire x1="23.495" y1="49.2125" x2="29.2125" y2="49.2125" width="0.254" layer="16"/>
-<wire x1="29.2125" y1="49.2125" x2="31.23" y2="51.23" width="0.254" layer="16"/>
+<contactref element="PCB1" pad="21"/>
+<wire x1="21.2725" y1="44.6659" x2="21.2725" y2="46.6725" width="0.254" layer="16"/>
+<wire x1="21.2725" y1="46.6725" x2="23.495" y2="48.895" width="0.254" layer="16"/>
+<wire x1="23.495" y1="48.895" x2="31.435" y2="48.895" width="0.254" layer="16"/>
+<wire x1="31.435" y1="48.895" x2="33.77" y2="51.23" width="0.254" layer="16"/>
 </signal>
 <signal name="CLK">
