File: MotorBoardPrototyp4_polyfuse.brd (EAGLE design)
At the start: 85 x 56 mm, 88 parts, among them IC1 OPA4340E, IC2 OPA4340E

Commit message: converted file format back to eagle version 6.6.0
Parts:
- C10: device rcl:C1812 -> rcl@1:C1812
Changed lines of the file:
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@@
 <?xml version="1.0" encoding="utf-8"?>
 <!DOCTYPE eagle SYSTEM "eagle.dtd">
-<eagle version="8.2.0">
+<eagle version="6.6.0">
 <drawing>
 <settings>
@@
 <pass name="Default">
 <param name="RoutingGrid" value="50mil"/>
-<param name="AutoGrid" value="1"/>
-<param name="Efforts" value="0"/>
-<param name="TopRouterVariant" value="1"/>
 <param name="tpViaShape" value="round"/>
-<param name="PrefDir.1" value="a"/>
+<param name="PrefDir.1" value="|"/>
 <param name="PrefDir.2" value="0"/>
 <param name="PrefDir.3" value="0"/>
@@
 <param name="PrefDir.14" value="0"/>
 <param name="PrefDir.15" value="0"/>
-<param name="PrefDir.16" value="a"/>
+<param name="PrefDir.16" value="-"/>
 <param name="cfVia" value="8"/>
 <param name="cfNonPref" value="5"/>
@@
 <element name="F7" library="SMD-Fuse" package="1812L050" value="POLY-FUSE" x="74.295" y="35.56" smashed="yes" rot="R270"/>
 <element name="F8" library="SMD-Fuse" package="1812L050" value="POLY-FUSE" x="74.295" y="48.26" smashed="yes" rot="R270"/>
-<element name="C10" library="rcl" library_urn="urn:adsk.eagle:library:334" package="C1812" value="" x="80.645" y="5.08" smashed="yes" rot="R270">
+<element name="C10" library="rcl@1" package="C1812" value="" x="80.645" y="5.08" smashed="yes" rot="R270">
 <attribute name="NAME" x="79.375" y="8.89" size="1.27" layer="25"/>
 <attribute name="VALUE" x="76.835" y="6.985" size="1.27" layer="27" rot="R270"/>
@@
 </board>
 </drawing>
-<compatibility>
-<note version="8.2" severity="warning">
-Since Version 8.2, Eagle supports online libraries. The ids
-of those online libraries will not be understood (or retained)
-with this version.
-</note>
-</compatibility>
 </eagle>
