File: MotorShield.sch (EAGLE design)
At the start: 119 parts, among them IC1 OPA4340E, IC2 OPA4340E, IC3 74HCT125D, X1 MSTBV2, X2 MSTBV8, X3 MSTBV8, X4 INPUTS, X5 BUTTON_LED, X6 DOTSTARS

Commit message: routed M1 to M4
Parts:
- F1, F2, F3, F4, F5, F6, F7, F8: value 1812L -> 1A
- LED1, LED2: device led:LEDCHIPLED_0603 -> led:LEDCHIP-LED0805
- LED11: device led:LEDCHIP-LED0603 -> led:LEDCHIPLED_0805
- LED12, LED13, LED14, LED15, LED3, LED4, LED5, LED6, LED7, LED8: device led:LEDCHIP-LED0603 -> led:LEDCHIP-LED0805
- R1, R10, R2, R41, R42, R43, R44, R45, R46, R47, R48, R49, R50, R51, R56: device rcl:R-EU_R0603 -> rcl:R-EU_R0805
Changed lines of the file:
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@@
 <class number="0" name="signal" width="0" drill="0">
 </class>
-<class number="1" name="motor 2A" width="0.4064" drill="0">
+<class number="1" name="motor 2A" width="0.8128" drill="0">
 </class>
 <class number="2" name="input 8A" width="2.54" drill="0">
@@
 <part name="PCB1" library="RASPBERRY_PI_GPIO" deviceset="RASPBERRY_PI_B+" device="_DIM"/>
 <part name="IC1" library="burr-brown" deviceset="OPA4340" device="E"/>
-<part name="IC2" library="burr-brown" deviceset="OPA4340" device="E"/>
-<part name="R1" library="rcl" deviceset="R-EU_" device="R0603" value="100m"/>
+<part name="IC2" library="burr-brown" deviceset="OPA4340" device="E" value="OPA4340E"/>
+<part name="R1" library="rcl" deviceset="R-EU_" device="R0805" value="100m"/>
 <part name="C1" library="eagle-ltspice" deviceset="C" device="" value="10nF"/>
 <part name="D1" library="diode" deviceset="DIODE-" device="DO214AA" value="200V/4A"/>
-<part name="R2" library="rcl" deviceset="R-EU_" device="R0603" value="100k"/>
+<part name="R2" library="rcl" deviceset="R-EU_" device="R0805" value="100k"/>
 <part name="R17" library="rcl" deviceset="R-EU_" device="R0805" value="27k"/>
 <part name="R18" library="rcl" deviceset="R-EU_" device="R0805" value="1k"/>
@@
 <part name="C4" library="eagle-ltspice" deviceset="C" device="" value="10nF"/>
 <part name="D4" library="diode" deviceset="DIODE-" device="DO214AA" value="200V/4A"/>
-<part name="R10" library="rcl" deviceset="R-EU_" device="R0603" value="100k"/>
+<part name="R10" library="rcl" deviceset="R-EU_" device="R0805" value="100k"/>
 <part name="R11" library="rcl" deviceset="R-EU_" device="R0805" value="10k"/>
 <part name="R12" library="rcl" deviceset="R-EU_" device="R0805" value="100m"/>
@@
 <part name="X6" library="con-wago255" deviceset="233-203" device="" value="DOTSTARS"/>
 <part name="GND4" library="supply1" deviceset="GND" device=""/>
-<part name="F1" library="ptc-littlefuse" deviceset="1812L" device=""/>
-<part name="F2" library="ptc-littlefuse" deviceset="1812L" device=""/>
-<part name="F3" library="ptc-littlefuse" deviceset="1812L" device=""/>
-<part name="F4" library="ptc-littlefuse" deviceset="1812L" device=""/>
-<part name="F5" library="ptc-littlefuse" deviceset="1812L" device=""/>
-<part name="F6" library="ptc-littlefuse" deviceset="1812L" device=""/>
-<part name="F7" library="ptc-littlefuse" deviceset="1812L" device=""/>
-<part name="F8" library="ptc-littlefuse" deviceset="1812L" device=""/>
-<part name="LED1" library="led" deviceset="LED" device="CHIPLED_0603" value="red"/>
-<part name="LED2" library="led" deviceset="LED" device="CHIPLED_0603" value="yellow"/>
-<part name="LED3" library="led" deviceset="LED" device="CHIP-LED0603" value="red"/>
-<part name="LED4" library="led" deviceset="LED" device="CHIP-LED0603" value="yellow"/>
-<part name="LED5" library="led" deviceset="LED" device="CHIP-LED0603" value="red"/>
-<part name="LED6" library="led" deviceset="LED" device="CHIP-LED0603" value="yellow"/>
-<part name="LED7" library="led" deviceset="LED" device="CHIP-LED0603" value="red"/>
-<part name="LED8" library="led" deviceset="LED" device="CHIP-LED0603" value="yellow"/>
+<part name="F1" library="ptc-littlefuse" deviceset="1812L" device="" value="1A"/>
+<part name="F2" library="ptc-littlefuse" deviceset="1812L" device="" value="1A"/>
+<part name="F3" library="ptc-littlefuse" deviceset="1812L" device="" value="1A"/>
+<part name="F4" library="ptc-littlefuse" deviceset="1812L" device="" value="1A"/>
+<part name="F5" library="ptc-littlefuse" deviceset="1812L" device="" value="1A"/>
+<part name="F6" library="ptc-littlefuse" deviceset="1812L" device="" value="1A"/>
+<part name="F7" library="ptc-littlefuse" deviceset="1812L" device="" value="1A"/>
+<part name="F8" library="ptc-littlefuse" deviceset="1812L" device="" value="1A"/>
+<part name="LED1" library="led" deviceset="LED" device="CHIP-LED0805" value="red"/>
+<part name="LED2" library="led" deviceset="LED" device="CHIP-LED0805" value="yellow"/>
+<part name="LED3" library="led" deviceset="LED" device="CHIP-LED0805" value="red"/>
+<part name="LED4" library="led" deviceset="LED" device="CHIP-LED0805" value="yellow"/>
+<part name="LED5" library="led" deviceset="LED" device="CHIP-LED0805" value="red"/>
+<part name="LED6" library="led" deviceset="LED" device="CHIP-LED0805" value="yellow"/>
+<part name="LED7" library="led" deviceset="LED" device="CHIP-LED0805" value="red"/>
+<part name="LED8" library="led" deviceset="LED" device="CHIP-LED0805" value="yellow"/>
 <part name="LED9" library="led" deviceset="LED" device="CHIP-LED0603" value="red"/>
 <part name="LED10" library="led" deviceset="LED" device="CHIP-LED0603" value="yellow"/>
-<part name="LED11" library="led" deviceset="LED" device="CHIP-LED0603" value="red"/>
-<part name="LED12" library="led" deviceset="LED" device="CHIP-LED0603" value="yellow"/>
-<part name="LED13" library="led" deviceset="LED" device="CHIP-LED0603" value="red"/>
-<part name="LED14" library="led" deviceset="LED" device="CHIP-LED0603" value="yellow"/>
-<part name="LED15" library="led" deviceset="LED" device="CHIP-LED0603" value="red"/>
+<part name="LED11" library="led" deviceset="LED" device="CHIPLED_0805" value="red"/>
+<part name="LED12" library="led" deviceset="LED" device="CHIP-LED0805" value="yellow"/>
+<part name="LED13" library="led" deviceset="LED" device="CHIP-LED0805" value="red"/>
+<part name="LED14" library="led" deviceset="LED" device="CHIP-LED0805" value="yellow"/>
+<part name="LED15" library="led" deviceset="LED" device="CHIP-LED0805" value="red"/>
 <part name="LED16" library="led" deviceset="LED" device="CHIP-LED0603" value="yellow"/>
-<part name="R41" library="rcl" deviceset="R-EU_" device="R0603" value="2k2"/>
-<part name="R42" library="rcl" deviceset="R-EU_" device="R0603" value="2k2"/>
-<part name="R43" library="rcl" deviceset="R-EU_" device="R0603" value="2k2"/>
-<part name="R44" library="rcl" deviceset="R-EU_" device="R0603" value="2k2"/>
-<part name="R45" library="rcl" deviceset="R-EU_" device="R0603" value="2k2"/>
-<part name="R46" library="rcl" deviceset="R-EU_" device="R0603" value="2k2"/>
-<part name="R47" library="rcl" deviceset="R-EU_" device="R0603" value="2k2"/>
-<part name="R48" library="rcl" deviceset="R-EU_" device="R0603" value="2k2"/>
-<part name="R49" library="rcl" deviceset="R-EU_" device="R0603" value="2k2"/>
-<part name="R50" library="rcl" deviceset="R-EU_" device="R0603" value="2k2"/>
-<part name="R51" library="rcl" deviceset="R-EU_" device="R0603" value="2k2"/>
+<part name="R41" library="rcl" deviceset="R-EU_" device="R0805" value="2k2"/>
+<part name="R42" library="rcl" deviceset="R-EU_" device="R0805" value="2k2"/>
+<part name="R43" library="rcl" deviceset="R-EU_" device="R0805" value="2k2"/>
+<part name="R44" library="rcl" deviceset="R-EU_" device="R0805" value="2k2"/>
+<part name="R45" library="rcl" deviceset="R-EU_" device="R0805" value="2k2"/>
+<part name="R46" library="rcl" deviceset="R-EU_" device="R0805" value="2k2"/>
+<part name="R47" library="rcl" deviceset="R-EU_" device="R0805" value="2k2"/>
+<part name="R48" library="rcl" deviceset="R-EU_" device="R0805" value="2k2"/>
+<part name="R49" library="rcl" deviceset="R-EU_" device="R0805" value="2k2"/>
+<part name="R50" library="rcl" deviceset="R-EU_" device="R0805" value="2k2"/>
+<part name="R51" library="rcl" deviceset="R-EU_" device="R0805" value="2k2"/>
 <part name="R52" library="rcl" deviceset="R-EU_" device="R0603" value="2k2"/>
 <part name="R53" library="rcl" deviceset="R-EU_" device="R0603" value="2k2"/>
 <part name="R54" library="rcl" deviceset="R-EU_" device="R0603" value="2k2"/>
 <part name="R55" library="rcl" deviceset="R-EU_" device="R0603" value="2k2"/>
-<part name="R56" library="rcl" deviceset="R-EU_" device="R0603" value="2k2"/>
+<part name="R56" library="rcl" deviceset="R-EU_" device="R0805" value="2k2"/>
 <part name="P+3" library="supply1" deviceset="+24V" device=""/>
 <part name="GND5" library="supply1" deviceset="GND" device=""/>

Commit message: placed parts for M5-M6
Parts:
- LED10, LED16, LED9: device led:LEDCHIP-LED0603 -> led:LEDCHIP-LED0805
- LED11: device led:LEDCHIPLED_0805 -> led:LEDCHIP-LED0805
- R52, R53, R54, R55: device rcl:R-EU_R0603 -> rcl:R-EU_R0805
Changed lines of the file:
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@@
 <part name="LED7" library="led" deviceset="LED" device="CHIP-LED0805" value="red"/>
 <part name="LED8" library="led" deviceset="LED" device="CHIP-LED0805" value="yellow"/>
-<part name="LED9" library="led" deviceset="LED" device="CHIP-LED0603" value="red"/>
-<part name="LED10" library="led" deviceset="LED" device="CHIP-LED0603" value="yellow"/>
-<part name="LED11" library="led" deviceset="LED" device="CHIPLED_0805" value="red"/>
+<part name="LED9" library="led" deviceset="LED" device="CHIP-LED0805" value="red"/>
+<part name="LED10" library="led" deviceset="LED" device="CHIP-LED0805" value="yellow"/>
+<part name="LED11" library="led" deviceset="LED" device="CHIP-LED0805" value="red"/>
 <part name="LED12" library="led" deviceset="LED" device="CHIP-LED0805" value="yellow"/>
 <part name="LED13" library="led" deviceset="LED" device="CHIP-LED0805" value="red"/>
 <part name="LED14" library="led" deviceset="LED" device="CHIP-LED0805" value="yellow"/>
 <part name="LED15" library="led" deviceset="LED" device="CHIP-LED0805" value="red"/>
-<part name="LED16" library="led" deviceset="LED" device="CHIP-LED0603" value="yellow"/>
+<part name="LED16" library="led" deviceset="LED" device="CHIP-LED0805" value="yellow"/>
 <part name="R41" library="rcl" deviceset="R-EU_" device="R0805" value="2k2"/>
 <part name="R42" library="rcl" deviceset="R-EU_" device="R0805" value="2k2"/>
@@
 <part name="R50" library="rcl" deviceset="R-EU_" device="R0805" value="2k2"/>
 <part name="R51" library="rcl" deviceset="R-EU_" device="R0805" value="2k2"/>
-<part name="R52" library="rcl" deviceset="R-EU_" device="R0603" value="2k2"/>
-<part name="R53" library="rcl" deviceset="R-EU_" device="R0603" value="2k2"/>
-<part name="R54" library="rcl" deviceset="R-EU_" device="R0603" value="2k2"/>
-<part name="R55" library="rcl" deviceset="R-EU_" device="R0603" value="2k2"/>
+<part name="R52" library="rcl" deviceset="R-EU_" device="R0805" value="2k2"/>
+<part name="R53" library="rcl" deviceset="R-EU_" device="R0805" value="2k2"/>
+<part name="R54" library="rcl" deviceset="R-EU_" device="R0805" value="2k2"/>
+<part name="R55" library="rcl" deviceset="R-EU_" device="R0805" value="2k2"/>
 <part name="R56" library="rcl" deviceset="R-EU_" device="R0805" value="2k2"/>
 <part name="P+3" library="supply1" deviceset="+24V" device=""/>

Commit message: routed op-amps
Parts:
- C10: value (none) -> 22uF
- T1, T2, T3, T4, T5, T6, T7, T8: value (none) -> FDN337N
- T9: value (none) -> BC847C
Connections:
- removed net +3,3V: IC1A.V+, IC2A.V+, PCB1.3V3@2
- net +3V3: now also IC1A.V+, IC2A.V+, PCB1.3V3@2
Changed lines of the file:
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@@
 <grid distance="0.1" unitdist="inch" unit="inch" style="lines" multiple="1" display="no" altdistance="0.01" altunitdist="inch" altunit="inch"/>
 <layers>
-<layer number="1" name="Top" color="4" fill="1" visible="yes" active="no"/>
-<layer number="16" name="Bottom" color="1" fill="1" visible="yes" active="no"/>
-<layer number="17" name="Pads" color="2" fill="1" visible="yes" active="no"/>
-<layer number="18" name="Vias" color="2" fill="1" visible="yes" active="no"/>
-<layer number="19" name="Unrouted" color="6" fill="1" visible="yes" active="no"/>
-<layer number="20" name="Dimension" color="15" fill="1" visible="yes" active="no"/>
-<layer number="21" name="tPlace" color="7" fill="1" visible="yes" active="no"/>
-<layer number="22" name="bPlace" color="7" fill="1" visible="yes" active="no"/>
-<layer number="23" name="tOrigins" color="15" fill="1" visible="yes" active="no"/>
-<layer number="24" name="bOrigins" color="15" fill="1" visible="yes" active="no"/>
-<layer number="25" name="tNames" color="7" fill="1" visible="yes" active="no"/>
-<layer number="26" name="bNames" color="7" fill="1" visible="yes" active="no"/>
-<layer number="27" name="tValues" color="7" fill="1" visible="yes" active="no"/>
-<layer number="28" name="bValues" color="7" fill="1" visible="yes" active="no"/>
+<layer number="1" name="Top" color="4" fill="1" visible="no" active="no"/>
+<layer number="16" name="Bottom" color="1" fill="1" visible="no" active="no"/>
+<layer number="17" name="Pads" color="2" fill="1" visible="no" active="no"/>
+<layer number="18" name="Vias" color="2" fill="1" visible="no" active="no"/>
+<layer number="19" name="Unrouted" color="6" fill="1" visible="no" active="no"/>
+<layer number="20" name="Dimension" color="15" fill="1" visible="no" active="no"/>
+<layer number="21" name="tPlace" color="7" fill="1" visible="no" active="no"/>
+<layer number="22" name="bPlace" color="7" fill="1" visible="no" active="no"/>
+<layer number="23" name="tOrigins" color="15" fill="1" visible="no" active="no"/>
+<layer number="24" name="bOrigins" color="15" fill="1" visible="no" active="no"/>
+<layer number="25" name="tNames" color="7" fill="1" visible="no" active="no"/>
+<layer number="26" name="bNames" color="7" fill="1" visible="no" active="no"/>
+<layer number="27" name="tValues" color="7" fill="1" visible="no" active="no"/>
+<layer number="28" name="bValues" color="7" fill="1" visible="no" active="no"/>
 <layer number="29" name="tStop" color="7" fill="3" visible="no" active="no"/>
 <layer number="30" name="bStop" color="7" fill="6" visible="no" active="no"/>
@@
 <layer number="35" name="tGlue" color="7" fill="4" visible="no" active="no"/>
 <layer number="36" name="bGlue" color="7" fill="5" visible="no" active="no"/>
-<layer number="37" name="tTest" color="7" fill="1" visible="yes" active="no"/>
-<layer number="38" name="bTest" color="7" fill="1" visible="yes" active="no"/>
+<layer number="37" name="tTest" color="7" fill="1" visible="no" active="no"/>
+<layer number="38" name="bTest" color="7" fill="1" visible="no" active="no"/>
 <layer number="39" name="tKeepout" color="4" fill="11" visible="no" active="no"/>
 <layer number="40" name="bKeepout" color="1" fill="11" visible="no" active="no"/>
@@
 <layer number="44" name="Drills" color="7" fill="1" visible="no" active="no"/>
 <layer number="45" name="Holes" color="7" fill="1" visible="no" active="no"/>
-<layer number="46" name="Milling" color="3" fill="1" visible="yes" active="no"/>
-<layer number="47" name="Measures" color="7" fill="1" visible="yes" active="no"/>
-<layer number="48" name="Document" color="7" fill="1" visible="yes" active="no"/>
-<layer number="49" name="Reference" color="7" fill="1" visible="yes" active="no"/>
-<layer number="50" name="dxf" color="7" fill="1" visible="yes" active="no"/>
-<layer number="51" name="tDocu" color="7" fill="1" visible="yes" active="no"/>
-<layer number="52" name="bDocu" color="7" fill="1" visible="yes" active="no"/>
-<layer number="53" name="tGND_GNDA" color="7" fill="9" visible="yes" active="no"/>
-<layer number="54" name="bGND_GNDA" color="1" fill="9" visible="yes" active="no"/>
-<layer number="56" name="wert" color="7" fill="1" visible="yes" active="no"/>
+<layer number="46" name="Milling" color="3" fill="1" visible="no" active="no"/>
+<layer number="47" name="Measures" color="7" fill="1" visible="no" active="no"/>
+<layer number="48" name="Document" color="7" fill="1" visible="no" active="no"/>
+<layer number="49" name="Reference" color="7" fill="1" visible="no" active="no"/>
+<layer number="50" name="dxf" color="7" fill="1" visible="no" active="no"/>
+<layer number="51" name="tDocu" color="7" fill="1" visible="no" active="no"/>
+<layer number="52" name="bDocu" color="7" fill="1" visible="no" active="no"/>
+<layer number="53" name="tGND_GNDA" color="7" fill="9" visible="no" active="no"/>
+<layer number="54" name="bGND_GNDA" color="1" fill="9" visible="no" active="no"/>
+<layer number="56" name="wert" color="7" fill="1" visible="no" active="no"/>
 <layer number="90" name="Modules" color="5" fill="1" visible="yes" active="yes"/>
 <layer number="91" name="Nets" color="2" fill="1" visible="yes" active="yes"/>
@@
 <part name="R39" library="rcl" deviceset="R-EU_" device="R0805" value="100k"/>
 <part name="R40" library="rcl" deviceset="R-EU_" device="R0805" value="10k"/>
-<part name="T1" library="zetex" deviceset="NMOSSOT23" device=""/>
-<part name="T2" library="zetex" deviceset="NMOSSOT23" device=""/>
-<part name="T3" library="zetex" deviceset="NMOSSOT23" device=""/>
-<part name="T4" library="zetex" deviceset="NMOSSOT23" device=""/>
-<part name="T5" library="zetex" deviceset="NMOSSOT23" device=""/>
-<part name="T6" library="zetex" deviceset="NMOSSOT23" device=""/>
-<part name="T7" library="zetex" deviceset="NMOSSOT23" device=""/>
-<part name="T8" library="zetex" deviceset="NMOSSOT23" device=""/>
-<part name="C10" library="rcl" deviceset="C-EU" device="C1812"/>
+<part name="T1" library="zetex" deviceset="NMOSSOT23" device="" value="FDN337N"/>
+<part name="T2" library="zetex" deviceset="NMOSSOT23" device="" value="FDN337N"/>
+<part name="T3" library="zetex" deviceset="NMOSSOT23" device="" value="FDN337N"/>
+<part name="T4" library="zetex" deviceset="NMOSSOT23" device="" value="FDN337N"/>
+<part name="T5" library="zetex" deviceset="NMOSSOT23" device="" value="FDN337N"/>
+<part name="T6" library="zetex" deviceset="NMOSSOT23" device="" value="FDN337N"/>
+<part name="T7" library="zetex" deviceset="NMOSSOT23" device="" value="FDN337N"/>
+<part name="T8" library="zetex" deviceset="NMOSSOT23" device="" value="FDN337N"/>
+<part name="C10" library="rcl" deviceset="C-EU" device="C1812" value="22uF"/>
 <part name="IC3" library="74xx-eu" deviceset="74*125" device="D" technology="HCT"/>
 <part name="X2" library="con-phoenix-508" deviceset="MSTBV8" device=""/>
@@
 <part name="GND1" library="supply1" deviceset="GND" device=""/>
 <part name="GND2" library="supply1" deviceset="GND" device=""/>
-<part name="T9" library="transistor" deviceset="*-NPN-" device="SOT23-BEC" technology="BC847C"/>
+<part name="T9" library="transistor" deviceset="*-NPN-" device="SOT23-BEC" technology="BC847C" value="BC847C"/>
 <part name="GND3" library="supply1" deviceset="GND" device=""/>
 <part name="X6" library="con-wago255" deviceset="233-203" device="" value="DOTSTARS"/>
@@
 <part name="GND7" library="supply1" deviceset="GND" device=""/>
 <part name="+3V2" library="supply1" deviceset="+3V3" device=""/>
+<part name="+3V3" library="supply1" deviceset="+3V3" device=""/>
+<part name="+3V4" library="supply1" deviceset="+3V3" device=""/>
+<part name="GND8" library="supply1" deviceset="GND" device=""/>
+<part name="GND9" library="supply1" deviceset="GND" device=""/>
 </parts>
 <sheets>
@@
 <instance part="GND7" gate="1" x="-12.7" y="30.48"/>
 <instance part="+3V2" gate="G$1" x="-12.7" y="96.52"/>
+<instance part="+3V3" gate="G$1" x="114.3" y="27.94"/>
+<instance part="+3V4" gate="G$1" x="215.9" y="25.4"/>
+<instance part="GND8" gate="1" x="114.3" y="0"/>
+<instance part="GND9" gate="1" x="215.9" y="-2.54"/>
 </instances>
 <busses>
@@
 <wire x1="114.3" y1="7.62" x2="114.3" y2="2.54" width="0.1524" layer="91"/>
 <label x="116.84" y="2.54" size="1.778" layer="95"/>
+<pinref part="GND8" gate="1" pin="GND"/>
 </segment>
 <segment>
@@
 <wire x1="215.9" y1="5.08" x2="215.9" y2="0" width="0.1524" layer="91"/>
 <label x="218.44" y="0" size="1.778" layer="95"/>
+<pinref part="GND9" gate="1" pin="GND"/>
 </segment>
 <segment>
@@
 </segment>
 </net>
-<net name="+3,3V" class="0">
-<segment>
-<pinref part="IC2" gate="A" pin="V+"/>
-<wire x1="215.9" y1="20.32" x2="215.9" y2="25.4" width="0.1524" layer="91"/>
-<label x="218.44" y="25.4" size="1.778" layer="95"/>
-</segment>
-<segment>
-<pinref part="IC1" gate="A" pin="V+"/>
-<wire x1="114.3" y1="22.86" x2="114.3" y2="27.94" width="0.1524" layer="91"/>
-<label x="116.84" y="27.94" size="1.778" layer="95"/>
-</segment>
-<segment>
-<pinref part="PCB1" gate="G$1" pin="3V3@2"/>
-<wire x1="-5.08" y1="66.04" x2="-12.7" y2="66.04" width="0.1524" layer="91"/>
-<label x="-20.32" y="66.04" size="1.778" layer="95"/>
-</segment>
-</net>
 <net name="N$2" class="1">
 <segment>
@@
 <wire x1="-12.7" y1="86.36" x2="-12.7" y2="93.98" width="0.1524" layer="91"/>
 </segment>
+<segment>
+<pinref part="PCB1" gate="G$1" pin="3V3@2"/>
+<wire x1="-5.08" y1="66.04" x2="-12.7" y2="66.04" width="0.1524" layer="91"/>
+<label x="-20.32" y="66.04" size="1.778" layer="95"/>
+</segment>
+<segment>
+<pinref part="IC2" gate="A" pin="V+"/>
+<pinref part="+3V4" gate="G$1" pin="+3V3"/>
+<wire x1="215.9" y1="20.32" x2="215.9" y2="22.86" width="0.1524" layer="91"/>
+</segment>
+<segment>
+<pinref part="IC1" gate="A" pin="V+"/>
+<pinref part="+3V3" gate="G$1" pin="+3V3"/>
+<wire x1="114.3" y1="22.86" x2="114.3" y2="25.4" width="0.1524" layer="91"/>
+</segment>
 </net>
 <net name="VCC" class="0">
@@
 </sheet>
 </sheets>
+<errors>
+</errors>
 </schematic>
 </drawing>
